Commit message: refactoring

File: body.urdf (robot description, URDF)
Before this commit: robot robot, 3 links, 2 joints
Links:
- removed link BackLeg
- removed link FrontLeg
- added link Backleg, mass 1; collision box size=1 1 1; visual box size=1 1 1
- added link Frontleg, mass 1; collision box size=1 1 1; visual box size=1 1 1
Joints:
- removed joint BackLeg_Torso
- added joint Torso_BackLeg: type revolute, parent Torso, child Backleg, origin xyz=1 0 1 rpy=0 0 0, axis 0 1 0, limit lower=-3.14159 upper=3.14159 effort=0.0 velocity=0.0
- joint Torso_FrontLeg: child FrontLeg -> Frontleg; origin xyz=1 0 -1 rpy=0 0 0 -> xyz=2 0 1 rpy=0 0 0

Commit message: quadruped

File: body.urdf (robot description, URDF)
Before this commit: robot robot, 3 links, 2 joints
Links:
- added link BackLowerleg, mass 1; collision box size=0.2 0.2 1; visual box size=0.2 0.2 1
- added link FrontLowerleg, mass 1; collision box size=0.2 0.2 1; visual box size=0.2 0.2 1
- added link LeftLowerleg, mass 1; collision box size=0.2 0.2 1; visual box size=0.2 0.2 1
- added link Leftleg, mass 1; collision box size=1 0.2 0.2; visual box size=1 0.2 0.2
- added link RightLowerleg, mass 1; collision box size=0.2 0.2 1; visual box size=0.2 0.2 1
- added link Rightleg, mass 1; collision box size=1 0.2 0.2; visual box size=1 0.2 0.2
- link Backleg: geometry collision box size=0.2 1 0.2; visual box size=0.2 1 0.2
- link Frontleg: geometry collision box size=0.2 1 0.2; visual box size=0.2 1 0.2
Joints:
- removed joint Torso_BackLeg
- removed joint Torso_FrontLeg
- added joint Backleg_BackLowerleg: type revolute, parent Backleg, child BackLowerleg, origin xyz=0 -1 0 rpy=0 0 0, axis 1 0 0, limit lower=-3.14159 upper=3.14159 effort=0.0 velocity=0.0
- added joint Frontleg_FrontLowerleg: type revolute, parent Frontleg, child FrontLowerleg, origin xyz=0 1 0 rpy=0 0 0, axis 1 0 0, limit lower=-3.14159 upper=3.14159 effort=0.0 velocity=0.0
- added joint Leftleg_LeftLowerleg: type revolute, parent Leftleg, child LeftLowerleg, origin xyz=-1 0 0 rpy=0 0 0, axis 0 1 0, limit lower=-3.14159 upper=3.14159 effort=0.0 velocity=0.0
- added joint Rightleg_RightLowerleg: type revolute, parent Rightleg, child RightLowerleg, origin xyz=1 0 0 rpy=0 0 0, axis 0 1 0, limit lower=-3.14159 upper=3.14159 effort=0.0 velocity=0.0
- added joint Torso_Backleg: type revolute, parent Torso, child Backleg, origin xyz=0 -0.5 1 rpy=0 0 0, axis 1 0 0, limit lower=-3.14159 upper=3.14159 effort=0.0 velocity=0.0
- added joint Torso_Frontleg: type revolute, parent Torso, child Frontleg, origin xyz=0 0.5 1 rpy=0 0 0, axis 1 0 0, limit lower=-3.14159 upper=3.14159 effort=0.0 velocity=0.0
- added joint Torso_Leftleg: type revolute, parent Torso, child Leftleg, origin xyz=-0.5 0 1 rpy=0 0 0, axis 0 1 0, limit lower=-3.14159 upper=3.14159 effort=0.0 velocity=0.0
- added joint Torso_Rightleg: type revolute, parent Torso, child Rightleg, origin xyz=0.5 0 1 rpy=0 0 0, axis 0 1 0, limit lower=-3.14159 upper=3.14159 effort=0.0 velocity=0.0

Commit message: final project phase1

File: body.urdf (robot description, URDF)
Before this commit: robot robot, 9 links, 8 joints
Links:
- removed link LeftLowerleg
- removed link Leftleg
- removed link RightLowerleg
- removed link Rightleg
- link Backleg: geometry collision box size=0.6 0.6 0.6; visual box size=0.6 0.6 0.6
- link Frontleg: geometry collision box size=0.2 0.2 0.2; visual box size=0.2 0.2 0.2
- link Torso: geometry collision box size=1.5 2 1; visual box size=1.5 2 1
Joints:
- removed joint Leftleg_LeftLowerleg
- removed joint Rightleg_RightLowerleg
- removed joint Torso_Leftleg
- removed joint Torso_Rightleg
- joint Backleg_BackLowerleg: origin xyz=0 -1 0 rpy=0 0 0 -> xyz=0 -0.5 -0.5 rpy=0 0 0
- joint Frontleg_FrontLowerleg: axis 1 0 0 -> -1 0 0; origin xyz=0 1 0 rpy=0 0 0 -> xyz=0 0 -0.5 rpy=0 0 0
- joint Torso_Backleg: origin xyz=0 -0.5 1 rpy=0 0 0 -> xyz=0 0 1 rpy=0 0 0

Commit message: ASSIGNMENT 6

File: body.urdf (robot description, URDF)
Before this commit: robot robot, 5 links, 4 joints
Links:
- removed link BackLowerleg
- removed link Backleg
- removed link FrontLowerleg
- removed link Frontleg
- removed link Torso
- added link Head, mass 1; collision box size=1 1 1; visual box size=1 1 1
- added link link0, mass 1; collision sphere radius=1.7102862782162553; visual sphere radius=1.7102862782162553
- added link link1, mass 1; collision cylinder length=1.1864015580919804 radius=1.245193797976902; visual cylinder length=1.1864015580919804 radius=1.245193797976902
- added link link2, mass 1; collision cylinder length=1.8502201984404887 radius=1.8720708001062114; visual cylinder length=1.8502201984404887 radius=1.8720708001062114
- added link link3, mass 1; collision cylinder length=1.9461018676910729 radius=1.197097679686683; visual cylinder length=1.9461018676910729 radius=1.197097679686683
- added link link4, mass 1; collision cylinder length=1.4414493789514182 radius=1.765794293342114; visual cylinder length=1.4414493789514182 radius=1.765794293342114
- added link link5, mass 1; collision sphere radius=1.3609992533883193; visual sphere radius=1.3609992533883193
- added link link6, mass 1; collision cylinder length=1.9369933078176897 radius=1.2265960175837307; visual cylinder length=1.9369933078176897 radius=1.2265960175837307
- added link link7, mass 1; collision box size=1.86653086959057 1.6740200614094731 1.0253092288735879; visual box size=1.86653086959057 1.6740200614094731 1.0253092288735879
- added link link8, mass 1; collision sphere radius=1.44807558423952; visual sphere radius=1.44807558423952
- added link link9, mass 1; collision sphere radius=1.0086060372130785; visual sphere radius=1.0086060372130785
Joints:
- removed joint Backleg_BackLowerleg
- removed joint Frontleg_FrontLowerleg
- removed joint Torso_Backleg
- removed joint Torso_Frontleg
- added joint Head_link0: type revolute, parent Head, child link0, origin xyz=-2 0 1 rpy=0 0 0, axis 0 0 1, limit lower=-3.14159 upper=3.14159 effort=0.0 velocity=0.0
- added joint link0_link1: type revolute, parent link0, child link1, origin xyz=-0.5 0 1 rpy=0 0 0, axis 0 0 1, limit lower=-3.14159 upper=3.14159 effort=0.0 velocity=0.0
- added joint link1_link2: type revolute, parent link1, child link2, origin xyz=-1.1864015580919804 0 0 rpy=0 0 0, axis 0 0 1, limit lower=-3.14159 upper=3.14159 effort=0.0 velocity=0.0
- added joint link2_link3: type revolute, parent link2, child link3, origin xyz=-1.8502201984404887 0 0 rpy=0 0 0, axis 0 0 1, limit lower=-3.14159 upper=3.14159 effort=0.0 velocity=0.0
- added joint link3_link4: type revolute, parent link3, child link4, origin xyz=-1.9461018676910729 0 0 rpy=0 0 0, axis 0 0 1, limit lower=-3.14159 upper=3.14159 effort=0.0 velocity=0.0
- added joint link4_link5: type revolute, parent link4, child link5, origin xyz=-1.4414493789514182 0 0 rpy=0 0 0, axis 0 0 1, limit lower=-3.14159 upper=3.14159 effort=0.0 velocity=0.0
- added joint link5_link6: type revolute, parent link5, child link6, origin xyz=-1.3609992533883193 0 0 rpy=0 0 0, axis 0 0 1, limit lower=-3.14159 upper=3.14159 effort=0.0 velocity=0.0
- added joint link6_link7: type revolute, parent link6, child link7, origin xyz=-1.9369933078176897 0 0 rpy=0 0 0, axis 0 0 1, limit lower=-3.14159 upper=3.14159 effort=0.0 velocity=0.0
- added joint link7_link8: type revolute, parent link7, child link8, origin xyz=-1.86653086959057 0 0 rpy=0 0 0, axis 0 0 1, limit lower=-3.14159 upper=3.14159 effort=0.0 velocity=0.0
- added joint link8_link9: type revolute, parent link8, child link9, origin xyz=-1.44807558423952 0 0 rpy=0 0 0, axis 0 0 1, limit lower=-3.14159 upper=3.14159 effort=0.0 velocity=0.0

Commit message: assignment 7 done

File: body.urdf (robot description, URDF)
Before this commit: robot robot, 11 links, 10 joints
Links:
- removed link Head
- removed link link3
- removed link link4
- removed link link5
- removed link link6
- removed link link7
- removed link link8
- removed link link9
- link link0: geometry collision box size=0.5620404076941705 0.2296378464009881 0.8134558433025307; visual box size=0.5620404076941705 0.2296378464009881 0.8134558433025307
- link link1: geometry collision box size=0.8071050574498323 0.8707873745002582 0.36622761764772194; visual box size=0.8071050574498323 0.8707873745002582 0.36622761764772194
- link link2: geometry collision box size=0.6713567582211156 0.1381732929702297 0.6132243551390095; visual box size=0.6713567582211156 0.1381732929702297 0.6132243551390095
Joints:
- removed joint Head_link0
- removed joint link2_link3
- removed joint link3_link4
- removed joint link4_link5
- removed joint link5_link6
- removed joint link6_link7
- removed joint link7_link8
- removed joint link8_link9
- joint link0_link1: axis 0 0 1 -> 0 1 0; origin xyz=-0.5 0 1 rpy=0 0 0 -> xyz=0 -0.28102020384708526 3 rpy=0 0 0
- joint link1_link2: axis 0 0 1 -> 1 0 0; origin xyz=-1.1864015580919804 0 0 rpy=0 0 0 -> xyz=-0.40355252872491615 -0.4353936872501291 0 rpy=0 0 0

Commit message: assignment 8 completed

File: body.urdf (robot description, URDF)
Before this commit: robot robot, 3 links, 2 joints
Links:
- added link link3, mass 1; collision box size=1.4193641228522977 1.437741136236781 1.855451736732372; visual box size=1.4193641228522977 1.437741136236781 1.855451736732372
- added link link4, mass 1; collision box size=1.3281555413942896 1.3346404640316147 1.4311407658665125; visual box size=1.3281555413942896 1.3346404640316147 1.4311407658665125
- added link link5, mass 1; collision box size=1.596734697973175 1.1931786941570774 1.177900231362671; visual box size=1.596734697973175 1.1931786941570774 1.177900231362671
- added link link6, mass 1; collision box size=1.1450451777324768 1.1932067053723352 1.9270145092262174; visual box size=1.1450451777324768 1.1932067053723352 1.9270145092262174
- added link link7, mass 1; collision box size=1.1334104382195567 1.4606857346835493 1.9130510847192432; visual box size=1.1334104382195567 1.4606857346835493 1.9130510847192432
- link link0: geometry collision box size=1.651351986334985 1.3945814265155008 1.3205253675283926; visual box size=1.651351986334985 1.3945814265155008 1.3205253675283926
- link link1: geometry collision box size=1.3349860129476125 1.4906224297188928 1.3499362822961212; visual box size=1.3349860129476125 1.4906224297188928 1.3499362822961212
- link link2: geometry collision box size=1.3021626224724958 1.3172827044783042 1.0907241593694064; visual box size=1.3021626224724958 1.3172827044783042 1.0907241593694064
Joints:
- added joint link2_link3: type revolute, parent link2, child link3, origin xyz=-0.6510813112362479 0 -0.5453620796847032 rpy=0 0 0, axis 1 0 0, limit lower=-3.14159 upper=3.14159 effort=0.0 velocity=0.0
- added joint link3_link4: type revolute, parent link3, child link4, origin xyz=-1.4193641228522977 0 0 rpy=0 0 0, axis 1 0 0, limit lower=-3.14159 upper=3.14159 effort=0.0 velocity=0.0
- added joint link4_link5: type revolute, parent link4, child link5, origin xyz=-1.3281555413942896 0 0 rpy=0 0 0, axis 1 0 0, limit lower=-3.14159 upper=3.14159 effort=0.0 velocity=0.0
- added joint link5_link6: type revolute, parent link5, child link6, origin xyz=-0.7983673489865875 -0.5965893470785387 0 rpy=0 0 0, axis 0 1 0, limit lower=-3.14159 upper=3.14159 effort=0.0 velocity=0.0
- added joint link6_link7: type revolute, parent link6, child link7, origin xyz=-0.5725225888662384 -0.5966033526861676 0 rpy=0 0 0, axis 1 0 0, limit lower=-3.14159 upper=3.14159 effort=0.0 velocity=0.0
- joint link0_link1: axis 0 1 0 -> 1 0 0; origin xyz=0 -0.28102020384708526 3 rpy=0 0 0 -> xyz=0.8256759931674925 0 5 rpy=0 0 0
- joint link1_link2: axis 1 0 0 -> 0 0 1; origin xyz=-0.40355252872491615 -0.4353936872501291 0 rpy=0 0 0 -> xyz=-0.6674930064738063 0 -0.6749681411480606 rpy=0 0 0

Commit message: FINAL

File: body.urdf (robot description, URDF)
Before this commit: robot robot, 8 links, 7 joints
Links:
- removed link link3
- removed link link4
- removed link link5
- removed link link6
- removed link link7
- link link0: geometry collision box size=0.6150761674340761 0.5321733370082746 0.9958009280713218; visual box size=0.6150761674340761 0.5321733370082746 0.9958009280713218
- link link1: geometry collision box size=0.6995730894676564 0.9776518095041434 0.550155880985586; visual box size=0.6995730894676564 0.9776518095041434 0.550155880985586
- link link2: geometry collision box size=0.9138493136093884 0.531924807422842 0.5189535441405086; visual box size=0.9138493136093884 0.531924807422842 0.5189535441405086
Joints:
- removed joint link2_link3
- removed joint link3_link4
- removed joint link4_link5
- removed joint link5_link6
- removed joint link6_link7
- joint link0_link1: origin xyz=0.8256759931674925 0 5 rpy=0 0 0 -> xyz=0.5 0 5 rpy=0 0 0
- joint link1_link2: axis 0 0 1 -> 0 1 0; origin xyz=-0.6674930064738063 0 -0.6749681411480606 rpy=0 0 0 -> xyz=0.3497865447338282 0.4888259047520717 0 rpy=0 0 0
