Commit message: Final changes

File: body0.urdf (robot description, URDF)
Before this commit: robot robot, 4 links, 3 joints
Links:
- link link0: geometry collision box size=0.5550242184096024 0.9350332930600187 0.6169267348587665; visual box size=0.5550242184096024 0.9350332930600187 0.6169267348587665
- link link1: geometry collision box size=0.684718673842597 0.6805140221682162 0.7531255272571132; visual box size=0.684718673842597 0.6805140221682162 0.7531255272571132
- link link2: geometry collision box size=0.830561083029109 0.6280572263507114 0.8576439428718199; visual box size=0.830561083029109 0.6280572263507114 0.8576439428718199
- link link3: geometry collision box size=0.6493328140625156 0.8279359490260615 0.5924964065643961; visual box size=0.6493328140625156 0.8279359490260615 0.5924964065643961
Joints:
- joint link0_link1: origin xyz=0 0 5.262520954972755 rpy=0 0 0 -> xyz=0 0 5.277512109204801 rpy=0 0 0
- joint link1_link2: origin xyz=0.4400374231078401 0 0.35568898085709777 rpy=0 0 0 -> xyz=0.3423593369212985 0 0.3765627636285566 rpy=0 0 0
- joint link2_link3: axis 1 0 0 -> 0 1 0; origin xyz=0.7736941500672652 0 0 rpy=0 0 0 -> xyz=0.4152805415145545 0.3140286131753557 0 rpy=0 0 0
